File: PCBDesign/NyxEagle/pcbWithuE.brd (EAGLE design)
At the start: 100 x 80 mm, 72 parts, among them IC1 STM32F10XCXT6, IC2 TCAN1051GVDRBRQ1, IC3 NUP2105, IC4 LM78L09ITPX_NOPB, IC5 DRV8304SRHAR

Commit message: Changed SPI Clock Edge setting to rising edge. Added Read Register function for drv8304 and added a function to read via SPI after reset of the controller, if the chip is locked.
Connections:
- net ENABLE: now also IC1.30
- net NFAULT: now also IC1.31
Routing:
- removed copper zone on layer 1, net SHC
Changed lines of the file:
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@@
 <wire x1="43.688" y1="53.594" x2="40.513" y2="56.769" width="0.2032" layer="16" curve="90"/>
 <wire x1="40.513" y1="56.769" x2="33.528" y2="56.769" width="0.2032" layer="16"/>
+<contactref element="IC1" pad="31"/>
+<wire x1="14.482" y1="16.946" x2="45.208" y2="44.479" width="0" layer="19" extent="1-1"/>
 </signal>
 <signal name="SDO">
@@
 <wire x1="47.908" y1="42.279" x2="47.92" y2="42.291" width="0.2032" layer="1" curve="-90"/>
 <wire x1="47.92" y1="42.291" x2="51.562" y2="42.291" width="0.2032" layer="1"/>
-<polygon width="0.0762" layer="1" isolate="1.016">
-</polygon>
 <wire x1="51.562" y1="42.291" x2="51.6382" y2="42.3672" width="0.3048" layer="1"/>
 <wire x1="58.928" y1="42.3672" x2="59.2582" y2="42.6974" width="0.3048" layer="1" curve="90"/>
@@
 <wire x1="38.989" y1="54.102" x2="33.655" y2="54.102" width="0.2032" layer="16"/>
 <wire x1="33.655" y1="54.102" x2="33.528" y2="54.229" width="0.2032" layer="16" curve="-90"/>
+<contactref element="IC1" pad="30"/>
+<wire x1="14.982" y1="16.946" x2="41.021" y2="44.45" width="0" layer="19" extent="1-1"/>
 </signal>
 <signal name="NSCS">
