File: PCBDesign/NyxEagle/pcbWithuE.sch (EAGLE design)
At the start: 72 parts, among them IC1 STM32F10XCXT6, IC2 TCAN1051GVDRBRQ1, IC3 NUP2105, IC4 LM78L09ITPX_NOPB, IC5 DRV8304SRHAR

Commit message: Changed SPI Clock Edge setting to rising edge. Added Read Register function for drv8304 and added a function to read via SPI after reset of the controller, if the chip is locked.
Connections:
- net ENABLE: now also IC1PORTA_H.PA9
- net NFAULT: now also IC1PORTA_H.PA10
Changed lines of the file:
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@@
+</segment>
+</net>
+<net name="ENABLE" class="0">
+<segment>
+<pinref part="IC1" gate="PORTA_H" pin="PA9"/>
+<wire x1="17.78" y1="86.36" x2="10.16" y2="86.36" width="0.1524" layer="91"/>
+<label x="2.54" y="86.36" size="1.778" layer="95"/>
+</segment>
+</net>
+<net name="NFAULT" class="0">
+<segment>
+<pinref part="IC1" gate="PORTA_H" pin="PA10"/>
+<wire x1="17.78" y1="83.82" x2="10.16" y2="83.82" width="0.1524" layer="91"/>
+<label x="2.54" y="83.82" size="1.778" layer="95"/>
 </segment>
 </net>
