File: PCBDesign/NyxEagle/pcbWithoutuE.brd (EAGLE design)
At the start: 69.9 x 73.4 mm, 35 parts, among them IC1 DRV8304SRHAR

Commit message: Added the DRV8304 component, which is used to configure the IC motor driver with the same name.
Parts:
- C2: value 1uF 16V -> 1uF 50V
Changed lines of the file:
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@@
 <attribute name="SPICEPREFIX" value="C" x="42.164" y="36.322" size="1.778" layer="27" display="off"/>
 </element>
-<element name="C2" library="rcl" library_urn="urn:adsk.eagle:library:334" package="C0805K" package3d_urn="urn:adsk.eagle:package:23681/2" value="1uF 16V" x="44.958" y="32.512" smashed="yes" rot="R180">
+<element name="C2" library="rcl" library_urn="urn:adsk.eagle:library:334" package="C0805K" package3d_urn="urn:adsk.eagle:package:23681/2" value="1uF 50V" x="44.958" y="32.512" smashed="yes" rot="R180">
 <attribute name="NAME" x="45.958" y="31.637" size="1.016" layer="25" rot="R180"/>
 <attribute name="SPICEPREFIX" value="C" x="44.958" y="32.512" size="1.778" layer="27" rot="R180" display="off"/>

Commit message: Update mul_s32_hiSR.h, queue.c, and 59 more files...
Parts:
- added C10, C11, C9: (no value), resistor:C0805
- added R11, R12, R13: (no value), resistor:R0805
- added T1, T10, T11, T12, T2, T3, T4, T5, T6, T7, T8, T9: TEST_POINT1593, ERIC:TURRET_TERMINAL_1593
- R10, R9: value (none) -> 0 Ohm; device rcl:R0201 -> resistor:R0603
- R8: value 0 -> 0 Ohm; device rcl:R0201 -> resistor:R0603
- moved INPUT 26.5 mm to (32.2, 10.5)
- moved C6 24.4 mm to (62.0, 54.1), turned to 180 degrees
- moved OUT3 24.0 mm to (73.6, 59.6)
- moved U$5 23.4 mm to (69.2, 55.4), turned to 270 degrees
- moved OUT2 22.0 mm to (73.6, 43.1)
- moved OUT1 22.0 mm to (73.6, 26.6)
- moved C7 21.4 mm to (62.0, 37.8), turned to 180 degrees
- moved U$3 20.4 mm to (69.2, 39.2), turned to 270 degrees
- moved GND 20.3 mm to (32.2, 15.4)
- moved U$2 19.7 mm to (69.2, 31.0), turned to 270 degrees
- moved C8 17.1 mm to (62.0, 20.7), turned to 180 degrees
- moved U$1 15.9 mm to (69.2, 22.9), turned to 270 degrees
- moved U$4 15.6 mm to (69.2, 47.3), turned to 270 degrees
- moved R6 14.7 mm to (49.1, 60.1)
- moved U$6 14.7 mm to (69.2, 63.6), turned to 270 degrees
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Connections:
- new net FED_SOA: ADCO.1, C9.1, R11.1
- new net FED_SOB: ADCO.2, C10.1, R12.2
- new net FED_SOC: ADCO.3, C11.1, R13.2
- net GHA: now also T4.1
- net GHB: now also T5.1
- net GHC: now also T6.1
- net GLA: now also T1.1
- net GLB: now also T2.1
- net GLC: now also T3.1
- net GND: now also C10.2, C11.2, C9.2
- net SHA: now also T10.1
- net SHB: now also T11.1
- net SHC: now also T12.1
- net SOA: now also R11.2; no longer ADCO.1
- net SOB: now also R12.1; no longer ADCO.2
- net SOC: now also R13.1; no longer ADCO.3
- net SPA: now also T7.1
- net SPB: now also T8.1
- net SPC: now also T9.1
Routing:
- net VM: track 211.3 -> 27.1 mm, vias 36 -> 0
- net GHC: track 75.3 -> 32.9 mm, vias 2 -> 1
- net GLA: track 63.9 -> 24.2 mm
- net GHB: track 57.0 -> 19.1 mm
- net SHA: track 63.2 -> 27.8 mm, vias 2 -> 0
- net SPA: track 59.8 -> 24.6 mm, vias 0 -> 2
- net SHB: track 56.8 -> 22.6 mm, vias 0 -> 2
- net SHC: track 60.7 -> 28.1 mm, vias 0 -> 2
- net SOB: track 39.1 -> 11.9 mm
- net SOA: track 37.7 -> 11.8 mm
- net AGND: track 30.2 -> 5.43 mm, vias 57 -> 1
- net SNA: track 38.3 -> 15.8 mm, vias 0 -> 2
- net GHA: track 49.4 -> 31.2 mm, vias 2 -> 0
- net SPC: track 44.5 -> 29.6 mm, vias 0 -> 2
- net GLB: track 40.2 -> 25.7 mm
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- removed copper zone on layer 1, net AGND
- removed copper zone on layer 16, net AGND
- removed copper zone on layer 16, net GND
- removed copper zone on layer 1, net SHA
- removed copper zone on layer 1, net SHB
- removed copper zone on layer 1, net SHC
- removed copper zone on layer 1, net SPA
- removed copper zone on layer 1, net SPB
- removed copper zone on layer 1, net SPC
- removed copper zone on layer 1, net VM
- removed copper zone on layer 16, net VM
Other:
- board text removed: "ADCO"
- board text removed: "C1"
- board text removed: "C2"
- board text removed: "C3"
- board text removed: "C4"
- board text removed: "C5"
- board text removed: "C6"
- board text removed: "C7"
- board text removed: "C8"
- board text removed: "GND"
- board text removed: "IC1"
- board text removed: "INPUT"
- board text removed: "OUT1"
- board text removed: "OUT2"
- board text removed: "OUT3"
- board text removed: "R1"
- board text removed: "R2"
- board text removed: "SPI"
